Commit message: Initial Moveit setup

File: tm20/urdf/tm20.urdf (robot description, URDF)
Before this commit: robot tm20, 8 links, 7 joints
Joints:
- joint joint_1: limit lower=-4.71 upper=4.71 effort=100 velocity=10 -> lower=-4.71 upper=4.71 effort=100 velocity=10.0
- joint joint_3: limit lower=-2.9 upper=2.9 effort=100 velocity=10 -> lower=-2.9 upper=2.9 effort=100 velocity=10.0
- joint joint_4: limit lower=-3.14 upper=3.14 effort=100 velocity=10 -> lower=-3.14 upper=3.14 effort=100 velocity=10.0
- joint joint_5: limit lower=-3.14 upper=3.14 effort=100 velocity=10 -> lower=-3.14 upper=3.14 effort=100 velocity=10.0
- joint joint_6: limit lower=-6.28 upper=6.28 effort=50 velocity=10 -> lower=-6.28 upper=6.28 effort=50 velocity=10.0

Commit message: update the static publisher

File: tm20/urdf/tm20.urdf (robot description, URDF)
Before this commit: robot tm20, 8 links, 7 joints
Joints:
- joint joint_6: axis 0 0 1 -> (none); limit lower=-6.28 upper=6.28 effort=50 velocity=10 -> (none); origin xyz=0 0.05 0 rpy=0 0 0 -> xyz=-0.012154 -0.0020165 0.12472 rpy=-0.0098957 -0.016364 1.5871; type revolute -> fixed

Commit message: Update tm20 package with working gripper and grey colors

File: tm20/urdf/tm20.urdf (robot description, URDF)
Before this commit: robot tm20, 8 links, 7 joints
Links:
- added link end_effector_based, mass 0.1; collision box size=0.05 0.12 0.05; visual mesh filename=package://tm20/meshes/end_effector_based.STL
- added link gripper_left, mass 0.05; collision box size=0.02 0.05 0.02; visual mesh filename=package://tm20/meshes/gripper_left.STL
- added link gripper_right, mass 0.05; collision box size=0.02 0.05 0.02; visual mesh filename=package://tm20/meshes/gripper_right.STL
- link link_3: mass 4.043 -> 6.177
- link link_5: mass 1.582 -> 1.58
- link link_6: mass 0.2 -> 0.044
Joints:
- added joint joint_7: type fixed, parent link_6, child end_effector_based, origin xyz=-0.00047 -0.0555 0 rpy=1.5702 -0.03148 -3.1237
- added joint joint_8: type prismatic, parent end_effector_based, child gripper_left, origin xyz=0 0.14178 0.01 rpy=3.1416 0 0, axis 1 0 0, limit lower=-0.02 upper=0 effort=50 velocity=0.1
- added joint joint_9: type prismatic, parent end_effector_based, child gripper_right, origin xyz=0 0.14178 -0.01 rpy=0 0 -3.1416, axis 1 0 0, limit lower=-0.02 upper=0 effort=50 velocity=0.1, mimic joint=joint_8 multiplier=1 offset=0
- joint joint_1: limit lower=-4.71 upper=4.71 effort=100 velocity=10.0 -> lower=-4.71 upper=4.71 effort=100 velocity=0.1; origin xyz=-0.04007 -0.00037 0.01545 rpy=1.5708 0 0.39147 -> xyz=-0.04007 -0.00037 0.01545 rpy=1.5708 0 -2.2375
- joint joint_2: limit lower=-3.14 upper=3.14 effort=100 velocity=10 -> lower=-3.14 upper=3.14 effort=100 velocity=0.1; origin xyz=0.14186 0.085 0 rpy=1.5708 -1.4804 -1.5708 -> xyz=0.18555 0.085 0 rpy=1.5708 -1.5658 -1.5708
- joint joint_3: axis 1 0 0 -> 0.999 0.039 0; limit lower=-2.9 upper=2.9 effort=100 velocity=10.0 -> lower=-2.9 upper=2.9 effort=100 velocity=0.1; origin xyz=0 0.6361 0 rpy=0.079313 1.5708 0 -> xyz=0 0.6361 0 rpy=-1.5708 1.5312 -1.5797
- joint joint_4: limit lower=-3.14 upper=3.14 effort=100 velocity=10.0 -> lower=-3.14 upper=3.14 effort=100 velocity=0.1; origin xyz=0 0.5271 0 rpy=3.1396 0 -3.1416 -> xyz=0 0.55558 0 rpy=3.1399 0 3.1416
- joint joint_5: limit lower=-3.14 upper=3.14 effort=100 velocity=10.0 -> lower=-3.14 upper=3.14 effort=100 velocity=0.1; origin xyz=-0.055141 0.060015 0 rpy=1.4876 0 -1.5708 -> xyz=0.060207 0.058537 0 rpy=1.5672 0 -1.5708
- joint joint_6: axis 0 0 1 -> (none); limit lower=-6.28 upper=6.28 effort=50 velocity=10.0 -> (none); origin xyz=-0.012154 -0.0020165 0.12472 rpy=-0.0098957 -0.016364 1.5871 -> xyz=-0.01348 -0.0014664 0.10695 rpy=0 -0.031485 -1.5886

Commit message: Revert "Update tm20 package with working gripper and grey colors"
This reverts commit 483e0740f4fe545c91f58ac5c4e3f49cd151ad02.

File: tm20/urdf/tm20.urdf (robot description, URDF)
Before this commit: robot tm20, 11 links, 10 joints
Links:
- removed link end_effector_based
- removed link gripper_left
- removed link gripper_right
- link link_3: mass 6.177 -> 4.043
- link link_5: mass 1.58 -> 1.582
- link link_6: mass 0.044 -> 0.2
Joints:
- removed joint joint_7
- removed joint joint_8
- removed joint joint_9
- joint joint_1: limit lower=-4.71 upper=4.71 effort=100 velocity=0.1 -> lower=-4.71 upper=4.71 effort=100 velocity=10.0; origin xyz=-0.04007 -0.00037 0.01545 rpy=1.5708 0 -2.2375 -> xyz=-0.04007 -0.00037 0.01545 rpy=1.5708 0 0.39147
- joint joint_2: limit lower=-3.14 upper=3.14 effort=100 velocity=0.1 -> lower=-3.14 upper=3.14 effort=100 velocity=10; origin xyz=0.18555 0.085 0 rpy=1.5708 -1.5658 -1.5708 -> xyz=0.14186 0.085 0 rpy=1.5708 -1.4804 -1.5708
- joint joint_3: axis 0.999 0.039 0 -> 1 0 0; limit lower=-2.9 upper=2.9 effort=100 velocity=0.1 -> lower=-2.9 upper=2.9 effort=100 velocity=10.0; origin xyz=0 0.6361 0 rpy=-1.5708 1.5312 -1.5797 -> xyz=0 0.6361 0 rpy=0.079313 1.5708 0
- joint joint_4: limit lower=-3.14 upper=3.14 effort=100 velocity=0.1 -> lower=-3.14 upper=3.14 effort=100 velocity=10.0; origin xyz=0 0.55558 0 rpy=3.1399 0 3.1416 -> xyz=0 0.5271 0 rpy=3.1396 0 -3.1416
- joint joint_5: limit lower=-3.14 upper=3.14 effort=100 velocity=0.1 -> lower=-3.14 upper=3.14 effort=100 velocity=10.0; origin xyz=0.060207 0.058537 0 rpy=1.5672 0 -1.5708 -> xyz=-0.055141 0.060015 0 rpy=1.4876 0 -1.5708
- joint joint_6: axis (none) -> 0 0 1; limit (none) -> lower=-6.28 upper=6.28 effort=50 velocity=10.0; origin xyz=-0.01348 -0.0014664 0.10695 rpy=0 -0.031485 -1.5886 -> xyz=-0.012154 -0.0020165 0.12472 rpy=-0.0098957 -0.016364 1.5871

Commit message: Updated robot with gripper and grey colors

File: tm20/urdf/tm20.urdf (robot description, URDF)
Before this commit: robot tm20, 8 links, 7 joints
Links:
- added link end_effector_based, mass 0.1; collision box size=0.05 0.12 0.05; visual mesh filename=package://tm20/meshes/end_effector_based.STL
- added link gripper_left, mass 0.05; collision box size=0.02 0.05 0.02; visual mesh filename=package://tm20/meshes/gripper_left.STL
- added link gripper_right, mass 0.05; collision box size=0.02 0.05 0.02; visual mesh filename=package://tm20/meshes/gripper_right.STL
- link link_3: mass 4.043 -> 6.177
- link link_5: mass 1.582 -> 1.58
- link link_6: mass 0.2 -> 0.044
Joints:
- added joint joint_7: type fixed, parent link_6, child end_effector_based, origin xyz=-0.00047 -0.0555 0 rpy=1.5702 -0.03148 -3.1237
- added joint joint_8: type prismatic, parent end_effector_based, child gripper_left, origin xyz=0 0.14178 0.01 rpy=3.1416 0 0, axis 1 0 0, limit lower=-0.02 upper=0 effort=50 velocity=0.1
- added joint joint_9: type prismatic, parent end_effector_based, child gripper_right, origin xyz=0 0.14178 -0.01 rpy=0 0 -3.1416, axis 1 0 0, limit lower=-0.02 upper=0 effort=50 velocity=0.1, mimic joint=joint_8 multiplier=1 offset=0
- joint joint_1: limit lower=-4.71 upper=4.71 effort=100 velocity=10 -> lower=-4.71 upper=4.71 effort=100 velocity=0.1; origin xyz=-0.04007 -0.00037 0.01545 rpy=1.5708 0 0.39147 -> xyz=-0.04007 -0.00037 0.01545 rpy=1.5708 0 -2.2375
- joint joint_2: limit lower=-3.14 upper=3.14 effort=100 velocity=10 -> lower=-3.14 upper=3.14 effort=100 velocity=0.1; origin xyz=0.14186 0.085 0 rpy=1.5708 -1.4804 -1.5708 -> xyz=0.18555 0.085 0 rpy=1.5708 -1.5658 -1.5708
- joint joint_3: axis 1 0 0 -> 0.999 0.039 0; limit lower=-2.9 upper=2.9 effort=100 velocity=10 -> lower=-2.9 upper=2.9 effort=100 velocity=0.1; origin xyz=0 0.6361 0 rpy=0.079313 1.5708 0 -> xyz=0 0.6361 0 rpy=-1.5708 1.5312 -1.5797
- joint joint_4: limit lower=-3.14 upper=3.14 effort=100 velocity=10 -> lower=-3.14 upper=3.14 effort=100 velocity=0.1; origin xyz=0 0.5271 0 rpy=3.1396 0 -3.1416 -> xyz=0 0.55558 0 rpy=3.1399 0 3.1416
- joint joint_5: limit lower=-3.14 upper=3.14 effort=100 velocity=10 -> lower=-3.14 upper=3.14 effort=100 velocity=0.1; origin xyz=-0.055141 0.060015 0 rpy=1.4876 0 -1.5708 -> xyz=0.060207 0.058537 0 rpy=1.5672 0 -1.5708
- joint joint_6: axis 0 0 1 -> (none); limit lower=-6.28 upper=6.28 effort=50 velocity=10 -> (none); origin xyz=0 0.05 0 rpy=0 0 0 -> xyz=-0.01348 -0.0014664 0.10695 rpy=0 -0.031485 -1.5886; type revolute -> fixed
